Commit message: Moveit File is added

File: src/arm_description/urdf/camera.urdf (robot description, URDF)
Before this commit: robot camera_sensor, 11 links, 10 joints
Links:
- link camera_head_link: geometry collision box size=0.02505 0.09 0.025; visual mesh filename=package://arm_description/meshes/collision/d435.stl

File: src/arm_description/urdf/panda.urdf.xacro (robot description, xacro)
@@ -29,5 +29,4 @@
         <origin xyz="0.0 0 0" rpy="0 0 0"/>
     </joint>
-    <virtual_joint name="fixed_frame" type="fixed" parent_frame="panda_link0" child_link="panda_link0" />
     <!--  -->
     <link name="panda_link1">

Commit message: CloudPoint2 works

File: src/arm_description/urdf/camera.urdf (robot description, URDF)
Before this commit: robot camera_sensor, 11 links, 10 joints
Links:
- removed link torso_link
- removed link world
- added link camera_base_link, mass 2.5; collision box size=0.15 0.10 0.06; collision cylinder length=1.0 radius=0.005
Joints:
- removed joint base_link_to_torso_link
- joint camera_head_joint: origin xyz=0 0.01 1.2 rpy=0 0.35 -0.15 -> xyz=-0.49 -0.5 1 rpy=0 0 0; parent torso_link -> camera_base_link

File: src/arm_description/urdf/panda.urdf.xacro (robot description, xacro)
@@ -29,4 +29,10 @@
         <origin xyz="0.0 0 0" rpy="0 0 0"/>
     </joint>
+    <!-- <link name="panda_mount"/>
+<joint name="panda_mount_joint" type="fixed">
+  <parent link="panda_mount"/>
+  <child link="panda_link0"/>
+  <origin xyz="0 0 0" rpy="0 0 0"/>
+</joint> -->
     <!--  -->
     <link name="panda_link1">
@@ -386,3 +392,151 @@
 </gazebo>
     <!--  -->
+<!-- Camera Module -->
+<link name="camera_base_link">
+    <visual name="holder">
+      <origin rpy="0 0 0" xyz="-0.5 -0.5 0.5"/>
+      <material name="LightGrey">
+        <color rgba="0.7 0.7 0.7 1.0"/>
+      </material>
+      <geometry>
+        <cylinder length="1.0" radius="0.005"/>
+      </geometry>
+    </visual>
+    <collision name="holder">
+      <origin rpy="0 0 0" xyz="-0.5 -0.5 0.5"/>
+      <geometry>
+        <cylinder length="1.0" radius="0.005"/>
+      </geometry>
+    </collision>
+    <visual name="base">
+      <origin rpy="0 0 0" xyz="-0.5 -0.5 0"/>
+      <material name="LightGrey">
+        <color rgba="0.7 0.7 0.7 1.0"/>
+      </material>
+      <geometry>
+        <box size="0.15 0.10 0.06"/>
+      </geometry>
+    </visual>
+    <collision name="base">
+      <origin rpy="0 0 0" xyz="-0.5 -0.5 0.0"/>
+      <geometry>
+        <box size="0.15 0.10 0.06"/>
+      </geometry>
+    </collision>
+    <inertial>
+      <origin xyz="-0.5 -0.5 0.50"/>
+      <mass value="2.5"/>
+      <inertia ixx="0.8" ixy="0.0" ixz="0.0" iyy="0.8" iyz="0.0" izz="0.8"/>
+    </inertial>
+  </link>
+  <!-- <link name ="world"/>
+  <joint name="world_to_camera_base_link" type="fixed">
+    <parent link="world"/>
+    <child link="camera_base_link"/>
+    <origin rpy="0 0 0" xyz="0 0 0"/>
+  </joint> -->
+<!-- Mount camera to Panda wrist -->
+<joint name="camera_mount_joint" type="fixed">
+  <parent link="panda_link0"/>
+  <child link="camera_base_link"/>
+  <origin xyz="0 0 0" rpy="0 0 0"/>
+</joint>
+  <link name="camera_head_link">
+    <visual>
+      <origin rpy="1.5707963267948966 0.0 1.5707963267948966" xyz="0 0 0"/>
+      <geometry>
+        <mesh filename="package://arm_description/meshes/collision/d435.stl"/>
+      </geometry>
+      <material name="aluminum">
+        <color rgba="0.5 0.5 0.5 1"/>
+      </material>
+    </visual>
+    <collision>
+      <origin rpy="0 0 0" xyz="0 0 0"/>
+      <geometry>
+        <box size="0.02505 0.09 0.025"/>
+      </geometry>
+    </collision>
+    <inertial>
+      <mass value="0.072"/>
+      <origin xyz="0 0 0"/>
+      <inertia ixx="0.003881243" ixy="0.0" ixz="0.0" iyy="0.000498940" iyz="0.0" izz="0.003879257"/>
+    </inertial>
+  </link>
+  <joint name="camera_head_joint" type="fixed">
+    <parent link="camera_base_link"/>
+    <child link="camera_head_link"/>
+    <origin rpy="0 0 0" xyz="-0.49 -0.5 1"/>
+  </joint>
+  <joint name="camera_head_depth_joint" type="fixed">
+    <origin rpy="0 0 0" xyz="0 0 0"/>
+    <parent link="camera_head_link"/>
+    <child link="camera_head_depth_frame"/>
+  </joint>
+  <link name="camera_head_depth_frame"/>
+  <joint name="camera_head_depth_optical_joint" type="fixed">
+    <origin rpy="-1.5707963267948966 0 -1.5707963267948966" xyz="0 0 0"/>
+    <parent link="camera_head_depth_frame"/>
+    <child link="camera_head_depth_optical_frame"/>
+  </joint>
+  <link name="camera_head_depth_optical_frame"/>
+  <joint name="camera_head_infra1_joint" type="fixed">
+    <origin rpy="0 0 0" xyz="0 0.0 0"/>
+    <parent link="camera_head_link"/>
+    <child link="camera_head_infra1_frame"/>
+  </joint>
+  <link name="camera_head_infra1_frame"/>
+  <joint name="camera_head_infra1_optical_joint" type="fixed">
+    <origin rpy="-1.5707963267948966 0 -1.5707963267948966" xyz="0 0 0"/>
+    <parent link="camera_head_infra1_frame"/>
+    <child link="camera_head_infra1_optical_frame"/>
+  </joint>
+  <link name="camera_head_infra1_optical_frame"/>
+  <joint name="camera_head_infra2_joint" type="fixed">
+    <origin rpy="0 0 0" xyz="0 -0.05 0"/>
+    <parent link="camera_head_link"/>
+    <child link="camera_head_infra2_frame"/>
+  </joint>
+  <link name="camera_head_infra2_frame"/>
+  <joint name="camera_head_infra2_optical_joint" type="fixed">
+    <origin rpy="-1.5707963267948966 0 -1.5707963267948966" xyz="0 0 0"/>
+    <parent link="camera_head_infra2_frame"/>
+    <child link="camera_head_infra2_optical_frame"/>
+  </joint>
+  <link name="camera_head_infra2_optical_frame"/>
+  <joint name="camera_head_color_joint" type="fixed">
+    <origin rpy="0 0 0" xyz="0 0.015 0"/>
+    <parent link="camera_head_link"/>
+    <child link="camera_head_color_frame"/>
+  </joint>
+  <link name="camera_head_color_frame"/>
+  <joint name="camera_head_color_optical_joint" type="fixed">
+    <origin rpy="-1.5707963267948966 0 -1.5707963267948966" xyz="0 0 0"/>
+    <parent link="camera_head_color_frame"/>
+    <child link="camera_head_color_optical_frame"/>
+  </joint>
+  <link name="camera_head_color_optical_frame"/>
+  <gazebo reference="camera_head_link">
+    <sensor name="camera_head" type="rgbd_camera">
+      <camera>
+        <horizontal_fov>1.5184</horizontal_fov>
+        <image>
+          <width>500</width>
+          <height>240</height>
+        </image>
+        <clip>
+          <near>0.05</near>
+          <far>3.0</far>
+        </clip>
+      </camera>
+      <always_on>1</always_on>
+      <gz_frame_id>camera_head_link</gz_frame_id>
+      <topic>camera_head</topic>
+      <update_rate>5</update_rate>
+      <visualize>true</visualize>
+    </sensor>
+  </gazebo>
+    <!-- <gazebo reference="panda_mount">
+  <static>true</static>
+</gazebo> -->
 </robot>
